File: hardware/analog/electro-load/electro-load/pwr.sch (KiCad schematic (older format))
At the start: 15 parts, among them J1 Conn_WallSocket_Earth, J2 Conn_WallSocket_Earth, U7 LM7805_TO220

Commit message: Added basic 3D model of amplifier encasing
Parts:
- removed J1: Conn_WallSocket_Earth, athir:Molex-KK-396-5277, symbol Connector:Barrel_Jack
- renumbered C16 to C29, C17 to C30, D1 to D3, D2 to D4, D3 to D5, D4 to D6, U7 to U14
Changed lines of the file:
@@
 EESchema Schematic File Version 4
-LIBS:electro-load-cache
 EELAYER 30 0
 EELAYER END
 $Descr A4 11693 8268
 encoding utf-8
-Sheet 6 6
+Sheet 5 5
 Title ""
 Date ""
@@
 Wire Wire Line
 	9125 4700 9050 4700
-$Comp
-L Connector:Barrel_Jack J1
-U 1 1 5E8304E0
-P 9425 4800
-F 0 "J1" H 9431 5225 50  0000 C CNN
-F 1 "Conn_WallSocket_Earth" H 10100 4900 50  0000 C CNN
-F 2 "athir:Molex-KK-396-5277" H 9125 4900 50  0001 C CNN
-F 3 "" H 9125 4900 50  0001 C CNN
-	1    9425 4800
-	-1   0    0    -1
-$EndComp
 Wire Wire Line
 	8550 4950 8875 4950
@@
 	8550 4700 8550 4625
 $Comp
-L Device:C_Small C17
+L Device:C_Small C30
 U 1 1 5E813619
 P 8550 4800
-F 0 "C17" H 8642 4846 50  0000 L CNN
+F 0 "C30" H 8642 4846 50  0000 L CNN
 F 1 "10u" H 8642 4755 50  0000 L CNN
 F 2 "Capacitor_SMD:C_0805_2012Metric" H 8550 4800 50  0001 C CNN
@@
 	8300 4700 8300 4625
 $Comp
-L Device:C_Small C16
+L Device:C_Small C29
 U 1 1 5E810C42
 P 8300 4800
-F 0 "C16" H 8392 4846 50  0000 L CNN
+F 0 "C29" H 8392 4846 50  0000 L CNN
 F 1 "100n" H 8200 4725 50  0000 L CNN
 F 2 "Capacitor_SMD:C_0603_1608Metric" H 8300 4800 50  0001 C CNN
@@
 AR Path="/5E80E014" Ref="#PWR?"  Part="1"
 AR Path="/5E8D69C1/5E80E014" Ref="#PWR0101"  Part="1"
-AR Path="/5E9F0954/5E80E014" Ref="#PWR0101"  Part="1"
-F 0 "#PWR0101" H 7850 4750 50  0001 C CNN
+AR Path="/5E9F0954/5E80E014" Ref="#PWR017"  Part="1"
+F 0 "#PWR017" H 7850 4750 50  0001 C CNN
 F 1 "GND" H 7855 4827 50  0000 C CNN
 F 2 "" H 7850 5000 50  0001 C CNN
@@
 $EndComp
 $Comp
-L Regulator_Linear:LM7805_TO220 U7
+L Regulator_Linear:LM7805_TO220 U14
 U 1 1 5E806D4B
 P 7850 4625
-F 0 "U7" H 7850 4867 50  0000 C CNN
+F 0 "U14" H 7850 4867 50  0000 C CNN
 F 1 "LM7805_TO220" H 7850 4776 50  0000 C CNN
 F 2 "Package_TO_SOT_THT:TO-220-3_Vertical" H 7850 4850 50  0001 C CIN
@@
 	5625 4775 6650 4775
 $Comp
-L Diode:1N914 D3
+L Diode:1N914 D5
 U 1 1 5E80EFD6
 P 6275 4625
-F 0 "D3" H 6275 4409 50  0000 C CNN
+F 0 "D5" H 6275 4409 50  0000 C CNN
 F 1 "1N5819" H 6275 4500 50  0000 C CNN
 F 2 "Diode_THT:D_DO-41_SOD81_P7.62mm_Horizontal" H 6275 4450 50  0001 C CNN
@@
 $EndComp
 $Comp
-L Diode:1N914 D4
+L Diode:1N914 D6
 U 1 1 5E80E8FD
 P 6275 4950
-F 0 "D4" H 6275 4734 50  0000 C CNN
+F 0 "D6" H 6275 4734 50  0000 C CNN
 F 1 "1N5819" H 6275 4825 50  0000 C CNN
 F 2 "Diode_THT:D_DO-41_SOD81_P7.62mm_Horizontal" H 6275 4775 50  0001 C CNN
@@
 $EndComp
 $Comp
-L Diode:1N914 D2
+L Diode:1N914 D4
 U 1 1 5E80E281
 P 5825 4950
-F 0 "D2" H 5825 4734 50  0000 C CNN
+F 0 "D4" H 5825 4734 50  0000 C CNN
 F 1 "1N5819" H 5825 4825 50  0000 C CNN
 F 2 "Diode_THT:D_DO-41_SOD81_P7.62mm_Horizontal" H 5825 4775 50  0001 C CNN
@@
 $EndComp
 $Comp
-L Diode:1N914 D1
+L Diode:1N914 D3
 U 1 1 5E80A819
 P 5825 4625
-F 0 "D1" H 5825 4409 50  0000 C CNN
+F 0 "D3" H 5825 4409 50  0000 C CNN
 F 1 "1N5819" H 5825 4500 50  0000 C CNN
 F 2 "Diode_THT:D_DO-41_SOD81_P7.62mm_Horizontal" H 5825 4450 50  0001 C CNN
@@
 $EndComp
 $Comp
-L power:VCC #PWR017
+L power:VCC #PWR015
 U 1 1 5E9F8E02
 P 3050 2775
-F 0 "#PWR017" H 3050 2625 50  0001 C CNN
+F 0 "#PWR015" H 3050 2625 50  0001 C CNN
 F 1 "VCC" H 3067 2948 50  0000 C CNN
 F 2 "" H 3050 2775 50  0001 C CNN
@@
 AR Path="/5E943757" Ref="#PWR?"  Part="1"
 AR Path="/5E8D69C1/5E943757" Ref="#PWR019"  Part="1"
-AR Path="/5E9F0954/5E943757" Ref="#PWR019"  Part="1"
-F 0 "#PWR019" H 7225 4775 50  0001 C CNN
+AR Path="/5E9F0954/5E943757" Ref="#PWR016"  Part="1"
+F 0 "#PWR016" H 7225 4775 50  0001 C CNN
 F 1 "GND" H 7230 4852 50  0000 C CNN
 F 2 "" H 7225 5025 50  0001 C CNN
@@
 	8225 4625 8225 4550
 $Comp
-L power:PWR_FLAG #FLG0101
+L power:PWR_FLAG #FLG02
 U 1 1 5E83DA07
 P 3050 4550
-F 0 "#FLG0101" H 3050 4625 50  0001 C CNN
+F 0 "#FLG02" H 3050 4625 50  0001 C CNN
 F 1 "PWR_FLAG" H 3050 4723 50  0000 C CNN
 F 2 "" H 3050 4550 50  0001 C CNN
@@
 $EndComp
 $Comp
-L power:PWR_FLAG #FLG0102
+L power:PWR_FLAG #FLG06
 U 1 1 5E83FFF2
 P 7400 4550
-F 0 "#FLG0102" H 7400 4625 50  0001 C CNN
+F 0 "#FLG06" H 7400 4625 50  0001 C CNN
 F 1 "PWR_FLAG" H 7400 4723 50  0000 C CNN
 F 2 "" H 7400 4550 50  0001 C CNN
@@
 AR Path="/5E94376D" Ref="C?"  Part="1"
 AR Path="/5E8D69C1/5E94376D" Ref="C9"  Part="1"
-AR Path="/5E9F0954/5E94376D" Ref="C9"  Part="1"
-F 0 "C9" H 7317 4821 50  0000 L CNN
+AR Path="/5E9F0954/5E94376D" Ref="C28"  Part="1"
+F 0 "C28" H 7317 4821 50  0000 L CNN
 F 1 "1000u" H 7317 4730 50  0000 L CNN
 F 2 "Capacitor_THT:CP_Radial_D10.0mm_P5.00mm" H 7225 4775 50  0001 C CNN
@@
 AR Path="/5E94375D" Ref="C?"  Part="1"
 AR Path="/5E8D69C1/5E94375D" Ref="C8"  Part="1"
-AR Path="/5E9F0954/5E94375D" Ref="C8"  Part="1"
-F 0 "C8" H 6775 4850 50  0000 L CNN
+AR Path="/5E9F0954/5E94375D" Ref="C27"  Part="1"
+F 0 "C27" H 6775 4850 50  0000 L CNN
 F 1 "1000u" H 6725 4725 50  0000 L CNN
 F 2 "Capacitor_THT:CP_Radial_D10.0mm_P5.00mm" H 6950 4775 50  0001 C CNN
@@
 AR Path="/5E96F498" Ref="C?"  Part="1"
 AR Path="/5E8D69C1/5E96F498" Ref="C1"  Part="1"
-AR Path="/5E9F0954/5E96F498" Ref="C1"  Part="1"
-F 0 "C1" H 8700 4875 50  0000 L CNN
+AR Path="/5E9F0954/5E96F498" Ref="C31"  Part="1"
+F 0 "C31" H 8700 4875 50  0000 L CNN
 F 1 "10u" H 8650 4750 50  0000 L CNN
 F 2 "Capacitor_THT:CP_Radial_D6.3mm_P2.50mm" H 8875 4800 50  0001 C CNN
@@
 Wire Wire Line
 	4925 5075 5175 5075
+$Comp
+L power:+5V #PWR?
+U 1 1 5E9F3114
+P 9125 4700
+F 0 "#PWR?" H 9125 4550 50  0001 C CNN
+F 1 "+5V" H 9140 4873 50  0000 C CNN
+F 2 "" H 9125 4700 50  0001 C CNN
+F 3 "" H 9125 4700 50  0001 C CNN
+	1    9125 4700
+	1    0    0    -1
+$EndComp
+$Comp
+L power:GND #PWR?
+U 1 1 5E9F392C
+P 9125 4950
+F 0 "#PWR?" H 9125 4700 50  0001 C CNN
+F 1 "GND" H 9130 4777 50  0000 C CNN
+F 2 "" H 9125 4950 50  0001 C CNN
+F 3 "" H 9125 4950 50  0001 C CNN
+	1    9125 4950
+	1    0    0    -1
+$EndComp
+Wire Wire Line
+	9125 4950 9125 4900
 $EndSCHEMATC

Commit message: Changed pin connections to/from lmv324 in order to avoid bird nesting. Widened traces for 5V and LOAD_CURRENT. Added four power resistors to the fab layer. Arranged left side analogs
Changed lines of the file:
@@
-$EndComp
-$Comp
-L power:PWR_FLAG #FLG?
-U 1 1 5E94378D
-P 2150 2725
-AR Path="/5E94378D" Ref="#FLG?"  Part="1"
-AR Path="/5E8D69C1/5E94378D" Ref="#FLG01"  Part="1"
-AR Path="/5E9F0954/5E94378D" Ref="#FLG01"  Part="1"
-F 0 "#FLG01" H 2150 2800 50  0001 C CNN
-F 1 "PWR_FLAG" H 2150 2898 50  0000 C CNN
-F 2 "" H 2150 2725 50  0001 C CNN
-F 3 "~" H 2150 2725 50  0001 C CNN
-	1    2150 2725
-	1    0    0    -1
-$EndComp
-Wire Wire Line
-	2150 2800 2150 2725
-$Comp
-L power:GND #PWR?
-U 1 1 5E94377D
-P 2150 2800
-AR Path="/5E94377D" Ref="#PWR?"  Part="1"
-AR Path="/5E8D69C1/5E94377D" Ref="#PWR014"  Part="1"
-AR Path="/5E9F0954/5E94377D" Ref="#PWR014"  Part="1"
-F 0 "#PWR014" H 2150 2550 50  0001 C CNN
-F 1 "GND" H 2155 2627 50  0000 C CNN
-F 2 "" H 2150 2800 50  0001 C CNN
-F 3 "" H 2150 2800 50  0001 C CNN
-	1    2150 2800
-	1    0    0    -1
 $EndComp
 $Comp
@@
 	4925 5075 5175 5075
 $Comp
-L power:+5V #PWR?
+L power:+5V #PWR0105
 U 1 1 5E9F3114
 P 9125 4700
-F 0 "#PWR?" H 9125 4550 50  0001 C CNN
+F 0 "#PWR0105" H 9125 4550 50  0001 C CNN
 F 1 "+5V" H 9140 4873 50  0000 C CNN
 F 2 "" H 9125 4700 50  0001 C CNN
@@
 $EndComp
 $Comp
-L power:GND #PWR?
+L power:GND #PWR0106
 U 1 1 5E9F392C
 P 9125 4950
-F 0 "#PWR?" H 9125 4700 50  0001 C CNN
+F 0 "#PWR0106" H 9125 4700 50  0001 C CNN
 F 1 "GND" H 9130 4777 50  0000 C CNN
 F 2 "" H 9125 4950 50  0001 C CNN
