File: hardware/analog/analog-main/analog0.sch (KiCad schematic (older format))
At the start: 15 parts, among them K1 SANYOU_SRD_Form_C, Q1 2N2222, U1 LMV321, U2 LMV321, U3 OPA549, U4 74HCT04

Commit message: Applied fixed symbol for OPA549
Configured all footprints
Parts:
- D1: footprint (none) -> LED_THT:LED_D5.0mm
- D2: footprint (none) -> Diode_THT:D_DO-35_SOD27_P7.62mm_Horizontal
- R2: footprint (none) -> Potentiometer_THT:Potentiometer_Bourns_3296W_Vertical
- U4: footprint (none) -> Package_SO:TSSOP-14_4.4x5mm_P0.65mm
Changed lines of the file:
@@
 F 0 "U4" H 9050 1867 50  0000 C CNN
 F 1 "74HCT04" H 9050 1776 50  0000 C CNN
-F 2 "" H 9050 1550 50  0001 C CNN
+F 2 "Package_SO:TSSOP-14_4.4x5mm_P0.65mm" H 9050 1550 50  0001 C CNN
 F 3 "https://assets.nexperia.com/documents/data-sheet/74HC_HCT04.pdf" H 9050 1550 50  0001 C CNN
 	1    9050 1550
@@
 F 0 "R2" V 8946 3150 50  0000 C CNN
 F 1 "10k POT" V 8855 3150 50  0000 C CNN
-F 2 "" H 8750 3150 50  0001 C CNN
+F 2 "Potentiometer_THT:Potentiometer_Bourns_3296W_Vertical" H 8750 3150 50  0001 C CNN
 F 3 "~" H 8750 3150 50  0001 C CNN
 	1    8750 3150
@@
 F 0 "D1" V 9996 1657 50  0000 R CNN
 F 1 "TEMP_LED" V 9905 1657 50  0000 R CNN
-F 2 "" V 9950 1725 50  0001 C CNN
+F 2 "LED_THT:LED_D5.0mm" V 9950 1725 50  0001 C CNN
 F 3 "~" V 9950 1725 50  0001 C CNN
 	1    9950 1725
@@
 F 0 "D2" H 10000 3591 50  0000 C CNN
 F 1 "D_Zener" H 10000 3500 50  0000 C CNN
-F 2 "" H 10000 3375 50  0001 C CNN
+F 2 "Diode_THT:D_DO-35_SOD27_P7.62mm_Horizontal" H 10000 3375 50  0001 C CNN
 F 3 "~" H 10000 3375 50  0001 C CNN
 	1    10000 3375

Commit message: Sorry future me
Parts:
- added C30: 4700u, Capacitor_THT:CP_Radial_D26.0mm_P10.00mm_SnapIn, symbol Device:CP
- added R?: 100R 1W+, Resistor_SMD:R_0603_1608Metric, symbol Device:R_Small
Connections:
- net GND: now also C30.2, R?.1
- net at K1.1, R2.2, U3.1 (VO)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: now also C30.1
- net at K1.4: now also R?.2
- net +36V renamed V+
- no-connect marks 1 -> 0
Changed lines of the file:
@@
 $Descr A4 11693 8268
 encoding utf-8
-Sheet 2 6
+Sheet 2 7
 Title ""
 Date ""
@@
 Connection ~ 6025 925
 $Comp
-L power:+36V #PWR08
-U 1 1 5E8FA61F
-P 8225 1950
-AR Path="/5E862B85/5E8FA61F" Ref="#PWR08"  Part="1"
-AR Path="/5E96F94C/5E8FA61F" Ref="#PWR?"  Part="1"
-F 0 "#PWR08" H 8225 1800 50  0001 C CNN
-F 1 "+36V" H 8240 2123 50  0000 C CNN
-F 2 "" H 8225 1950 50  0001 C CNN
-F 3 "" H 8225 1950 50  0001 C CNN
-	1    8225 1950
-	1    0    0    -1
-$EndComp
-$Comp
 L Relay:SANYOU_SRD_Form_C K1
 U 1 1 5E8FE364
@@
 $EndComp
 Wire Wire Line
-	9700 2525 9100 2525
+	9700 2525 9300 2525
 Connection ~ 9100 2525
 $Comp
@@
 	1    0    0    -1
 $EndComp
-NoConn ~ 10300 2625
 $Comp
 L Device:D_Zener D2
@@
 	7050 3150 6625 3150
 Connection ~ 6625 3150
-Text HLabel 10800 2425 2    50   Output ~ 0
+Text HLabel 10825 2425 2    50   Output ~ 0
 OUT_0+
+$Comp
+L Device:CP C?
+U 1 1 5EBCEB41
+P 9300 2750
+AR Path="/5EBAB32F/5EBCEB41" Ref="C?"  Part="1"
+AR Path="/5E862B85/5EBCEB41" Ref="C30"  Part="1"
+F 0 "C30" H 9418 2796 50  0000 L CNN
+F 1 "4700u" H 9418 2705 50  0000 L CNN
+F 2 "Capacitor_THT:CP_Radial_D26.0mm_P10.00mm_SnapIn" H 9338 2600 50  0001 C CNN
+F 3 "~" H 9300 2750 50  0001 C CNN
+	1    9300 2750
+	1    0    0    -1
+$EndComp
+Wire Wire Line
+	9300 2600 9300 2525
+Connection ~ 9300 2525
+Wire Wire Line
+	9300 2525 9100 2525
+$Comp
+L power:GND #PWR0109
+U 1 1 5EBD1EA5
+P 9300 3000
+AR Path="/5E862B85/5EBD1EA5" Ref="#PWR0109"  Part="1"
+AR Path="/5E96F94C/5EBD1EA5" Ref="#PWR?"  Part="1"
+F 0 "#PWR0109" H 9300 2750 50  0001 C CNN
+F 1 "GND" H 9305 2827 50  0000 C CNN
+F 2 "" H 9300 3000 50  0001 C CNN
+F 3 "" H 9300 3000 50  0001 C CNN
+	1    9300 3000
+	1    0    0    -1
+$EndComp
+Wire Wire Line
+	9300 2900 9300 3000
+Text Label 8225 1950 2    50   ~ 0
+AN0_VCC
+$Comp
+L Device:R_Small R?
+U 1 1 5EBF84B9
+P 10525 2625
+AR Path="/5E862B85/5EBF84B9" Ref="R?"  Part="1"
+AR Path="/5E96F94C/5EBF84B9" Ref="R?"  Part="1"
+F 0 "R?" V 10329 2625 50  0000 C CNN
+F 1 "100R 1W+" V 10420 2625 50  0000 C CNN
+F 2 "Resistor_SMD:R_0603_1608Metric" H 10525 2625 50  0001 C CNN
+F 3 "~" H 10525 2625 50  0001 C CNN
+	1    10525 2625
+	0    1    1    0
+$EndComp
+Wire Wire Line
+	10425 2625 10300 2625
+$Comp
+L power:GND #PWR?
+U 1 1 5EBFABE3
+P 10725 2700
+F 0 "#PWR?" H 10725 2450 50  0001 C CNN
+F 1 "GND" H 10730 2527 50  0000 C CNN
+F 2 "" H 10725 2700 50  0001 C CNN
+F 3 "" H 10725 2700 50  0001 C CNN
+	1    10725 2700
+	1    0    0    -1
+$EndComp
+Wire Wire Line
+	10725 2700 10725 2625
+Wire Wire Line
+	10725 2625 10625 2625
 $EndSCHEMATC
