File: hardware/analog/analog-main/current.sch (KiCad schematic (older format))
At the start: 42 parts, among them K3 SANYOU_SRD_Form_C, K4 SANYOU_SRD_Form_C, K5 SANYOU_SRD_Form_C, K6 SANYOU_SRD_Form_C, Q3 2N2222, Q4 2N2222, Q5 2N2222, Q6 2N2222, U17 MAX4239AUT, U18 MAX4239AUT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

Commit message: Applied fixed symbol for OPA549
Configured all footprints
Parts:
- D5, D6, D7, D8: footprint (none) -> Diode_THT:D_DO-35_SOD27_P7.62mm_Horizontal
- R19, R20, R21, R24, R25, R27, R32, R33, R34, R37, R38, R40: footprint (none) -> Resistor_SMD:R_0603_1608Metric
Changed lines of the file:
@@
 F 0 "D7" H 6350 6191 50  0000 C CNN
 F 1 "D_Zener" H 6350 6100 50  0000 C CNN
-F 2 "" H 6350 5975 50  0001 C CNN
+F 2 "Diode_THT:D_DO-35_SOD27_P7.62mm_Horizontal" H 6350 5975 50  0001 C CNN
 F 3 "~" H 6350 5975 50  0001 C CNN
 	1    6350 5975
@@
 F 0 "R33" V 8200 5225 50  0000 C CNN
 F 1 "10R 1%" V 8275 5225 50  0000 C CNN
-F 2 "" H 8200 5225 50  0001 C CNN
+F 2 "Resistor_SMD:R_0603_1608Metric" H 8200 5225 50  0001 C CNN
 F 3 "~" H 8200 5225 50  0001 C CNN
 	1    8200 5225
@@
 F 0 "R32" V 8200 5025 50  0000 C CNN
 F 1 "10m 1%" V 8125 5025 50  0000 C CNN
-F 2 "" H 8200 5025 50  0001 C CNN
+F 2 "Resistor_SMD:R_0603_1608Metric" H 8200 5025 50  0001 C CNN
 F 3 "~" H 8200 5025 50  0001 C CNN
 	1    8200 5025
@@
 F 0 "R37" V 8654 4925 50  0000 C CNN
 F 1 "6k8 1%" V 8745 4925 50  0000 C CNN
-F 2 "" H 8850 4925 50  0001 C CNN
+F 2 "Resistor_SMD:R_0603_1608Metric" H 8850 4925 50  0001 C CNN
 F 3 "~" H 8850 4925 50  0001 C CNN
 	1    8850 4925
@@
 F 0 "R38" V 9004 4925 50  0000 C CNN
 F 1 "2k2 1%" V 9095 4925 50  0000 C CNN
-F 2 "" H 9200 4925 50  0001 C CNN
+F 2 "Resistor_SMD:R_0603_1608Metric" H 9200 4925 50  0001 C CNN
 F 3 "~" H 9200 4925 50  0001 C CNN
 	1    9200 4925
@@
 F 0 "R40" V 10029 5025 50  0000 C CNN
 F 1 "3k 1%" V 10120 5025 50  0000 C CNN
-F 2 "" H 10225 5025 50  0001 C CNN
+F 2 "Resistor_SMD:R_0603_1608Metric" H 10225 5025 50  0001 C CNN
 F 3 "~" H 10225 5025 50  0001 C CNN
 	1    10225 5025
@@
 F 0 "D8" H 7750 7116 50  0000 C CNN
 F 1 "D_Zener" H 7750 7025 50  0000 C CNN
-F 2 "" H 7750 6900 50  0001 C CNN
+F 2 "Diode_THT:D_DO-35_SOD27_P7.62mm_Horizontal" H 7750 6900 50  0001 C CNN
 F 3 "~" H 7750 6900 50  0001 C CNN
 	1    7750 6900
@@
 F 0 "R34" V 8400 5950 50  0000 C CNN
 F 1 "10k 1%" V 8475 5950 50  0000 C CNN
-F 2 "" H 8400 5950 50  0001 C CNN
+F 2 "Resistor_SMD:R_0603_1608Metric" H 8400 5950 50  0001 C CNN
 F 3 "~" H 8400 5950 50  0001 C CNN
 	1    8400 5950
@@
 F 0 "D5" H 2025 3866 50  0000 C CNN
 F 1 "D_Zener" H 2025 3775 50  0000 C CNN
-F 2 "" H 2025 3650 50  0001 C CNN
+F 2 "Diode_THT:D_DO-35_SOD27_P7.62mm_Horizontal" H 2025 3650 50  0001 C CNN
 F 3 "~" H 2025 3650 50  0001 C CNN
 	1    2025 3650
@@
 F 0 "R20" V 3875 2900 50  0000 C CNN
 F 1 "10R 1%" V 3950 2900 50  0000 C CNN
-F 2 "" H 3875 2900 50  0001 C CNN
+F 2 "Resistor_SMD:R_0603_1608Metric" H 3875 2900 50  0001 C CNN
 F 3 "~" H 3875 2900 50  0001 C CNN
 	1    3875 2900
@@
 F 0 "R19" V 3875 2700 50  0000 C CNN
 F 1 "10m 1%" V 3800 2700 50  0000 C CNN
-F 2 "" H 3875 2700 50  0001 C CNN
+F 2 "Resistor_SMD:R_0603_1608Metric" H 3875 2700 50  0001 C CNN
 F 3 "~" H 3875 2700 50  0001 C CNN
 	1    3875 2700
@@
 F 0 "R24" V 4329 2600 50  0000 C CNN
 F 1 "6k8 1%" V 4420 2600 50  0000 C CNN
-F 2 "" H 4525 2600 50  0001 C CNN
+F 2 "Resistor_SMD:R_0603_1608Metric" H 4525 2600 50  0001 C CNN
 F 3 "~" H 4525 2600 50  0001 C CNN
 	1    4525 2600
@@
 F 0 "R25" V 4679 2600 50  0000 C CNN
 F 1 "2k2 1%" V 4770 2600 50  0000 C CNN
-F 2 "" H 4875 2600 50  0001 C CNN
+F 2 "Resistor_SMD:R_0603_1608Metric" H 4875 2600 50  0001 C CNN
 F 3 "~" H 4875 2600 50  0001 C CNN
 	1    4875 2600
@@
 F 0 "R27" V 5704 2700 50  0000 C CNN
 F 1 "3k 1%" V 5795 2700 50  0000 C CNN
-F 2 "" H 5900 2700 50  0001 C CNN
+F 2 "Resistor_SMD:R_0603_1608Metric" H 5900 2700 50  0001 C CNN
 F 3 "~" H 5900 2700 50  0001 C CNN
 	1    5900 2700
@@
 F 0 "D6" H 3425 4791 50  0000 C CNN
 F 1 "D_Zener" H 3425 4700 50  0000 C CNN
-F 2 "" H 3425 4575 50  0001 C CNN
+F 2 "Diode_THT:D_DO-35_SOD27_P7.62mm_Horizontal" H 3425 4575 50  0001 C CNN
 F 3 "~" H 3425 4575 50  0001 C CNN
 	1    3425 4575
@@
 F 0 "R21" V 4075 3625 50  0000 C CNN
 F 1 "10k 1%" V 4150 3625 50  0000 C CNN
-F 2 "" H 4075 3625 50  0001 C CNN
+F 2 "Resistor_SMD:R_0603_1608Metric" H 4075 3625 50  0001 C CNN
 F 3 "~" H 4075 3625 50  0001 C CNN
 	1    4075 3625

Commit message: Sorry future me
Parts:
- removed R26: 1k, Resistor_SMD:R_0603_1608Metric, symbol Device:R_Small
- removed R27: 3k 1%, Resistor_SMD:R_0603_1608Metric, symbol Device:R_Small
- removed U18: MAX4239AUT, Package_TO_SOT_SMD:SOT-23-6, symbol Amplifier_Operational:MAX4239AUT
- added RV1: 15k pot, symbol Device:R_POT_TRIM
- R19, R32: value 10m 1% -> 100m 1%
- R20, R33: value 10R 1% -> 5R 1%
- R22: value 100R -> 10k 1%
- R23: value 1k -> 1k 1%
- R24: value 6k8 1% -> 33k 1%
- R25: value 2k2 1% -> 1k 1%
Connections:
- net -5V: no longer U17.2 (V-)
- net CUR_MEAS_0: now also U17.1, RV1.3
- net GND: now also R25.1, U17.2 (V-)
- net at R22.1, U17.3 (+): now also R25.2
- net at R24.1: now also RV1.2; no longer R25.2
- no-connect marks 0 -> 1
Other:
- note removed: "x 10 x 4"
- moved on the sheet: R19, R20, R22
